File: COUPON_SMA_THRU_v1/COUPON_SMA_THRU_v1.kicad_pcb (KiCad board)
At the start: 4 copper layers, 62.8 x 22 mm, 4 parts, among them J1 Conn_Coaxial, J2 Conn_Coaxial, J3 Conn_Coaxial, J4 Conn_Coaxial

Commit message: Stackup edit
Parts:
- J1, J2, J3, J4: footprint Custom:SMA_Custom -> Project:Conn_SMA
